File: CM4_Carrier_Board/GPIO.kicad_sch (KiCad schematic)
At the start: 1 part, among them J6 Conn_02x20_Odd_Even

Commit message: Assignement des empreintes et début du PCB
Parts:
- J6: footprint (none) -> Connector_PinHeader_2.54mm:PinHeader_2x20_P2.54mm_Vertical
Changed lines of the file:
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@@
 			)
 		)
-		(property "Footprint" ""
+		(property "Footprint" "Connector_PinHeader_2.54mm:PinHeader_2x20_P2.54mm_Vertical"
 			(at 111.76 95.25 0)
 			(hide yes)
