File: CM4_Carrier_Board/bloc_USB_sch.kicad_sch (KiCad schematic)
At the start: 2 parts, among them J7 USB_A, U3 USBLC6-2SC6

Commit message: Assignement des empreintes et début du PCB
Parts:
- J7: footprint (none) -> Connector_USB:USB_A_Wuerth_614004134726_Horizontal
Changed lines of the file:
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@@
 			)
 		)
-		(property "Footprint" ""
+		(property "Footprint" "Connector_USB:USB_A_Wuerth_614004134726_Horizontal"
 			(at 68.58 59.69 0)
 			(hide yes)
